File: Schematic/Switch_Toggler/Switch_Toggler.sch (KiCad schematic (older format))
At the start: 30 parts, among them J1 AUTO_250, Q1 IRF540N, Q2 IRF540N, Q3 BC549, Q4 BC549, SW1 BUT_UP, SW2 BUT_DOWN, SW3 PWR_SW, U1 LM7805_TO220, U2 ATtiny85-20PU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

Commit message: Turned on clock point, minute support, new 2min max, better button hold timer interaction
Parts:
- U3: symbol my_library:TM1637 -> Switch_Toggler-rescue:TM1637-my_library
Changed lines of the file:
@@
 	9300 2950 9300 2800
 $Comp
-L my_library:TM1637 U3
+L Switch_Toggler-rescue:TM1637-my_library U3
 U 1 1 5F57E922
 P 4500 1500
